Commit message: stable

File: wallbe/description/lidar.urdf.xacro (robot description, xacro)
@@ -5,11 +5,11 @@
         <parent link="base_link"/>
         <child link="lidar_frame"/>
-        <origin xyz="0.1263 0.045 0" rpy="0 0 0"/>
+        <origin xyz="0.09 0 0" rpy="0 0 0"/>
     </joint>
     <link name="lidar_frame">
         <visual>
-            <origin xyz="0.0 0 0.1" rpy="${PI/2} 0 -${PI/2}"/>
+            <origin xyz="0.0 0 0.1" rpy="0 0 0"/>
             <geometry>
-                <mesh filename="package://wallBE/meshes/lidar.STL" scale="0.001 0.001 0.001"/>
+                <cylinder length="0.03" radius="0.02"/>
             </geometry>
             <material name="blue"/>

File: wallbe/description/robot.urdf.xacro (robot description, xacro)
@@ -1,7 +1,8 @@
 <?xml version="1.0"?>
 <robot xmlns:xacro="http://www.ros.org/wiki/xacro"  name="robot">
-    <xacro:include filename="materials.xacro" />
-    <xacro:include filename="robot_core.xacro" />
-    <!-- <xacro:include filename="lidar.xacro" /> -->
     <xacro:include filename="ros2_control.xacro" />
+    <xacro:include filename="materials.urdf.xacro" />
+    <xacro:include filename="robot_core.urdf.xacro" />
+    <xacro:include filename="lidar.urdf.xacro" />
+    <xacro:include filename="imu.urdf.xacro" />
 </robot>
