Commit message: add new node for serial

File: wallbe/description/imu.urdf.xacro (robot description, xacro)
@@ -4,10 +4,10 @@
         <parent link="base_link"/>
         <child link="imu_frame"/>
-        <origin xyz="0.09 0 0.081425" rpy="0 0 0"/>
+        <origin xyz="0.16 0 0.081425" rpy="0 0 0"/>
     </joint>
     <link name="imu_frame">
         <visual>
             <geometry>
-                <box size="0.0363 0.01755 0.005425"/>
+                <box size="0.024 0.012 0.005425"/>
             </geometry>
             <material name="green"/>

File: wallbe/description/lidar.urdf.xacro (robot description, xacro)
@@ -5,5 +5,5 @@
         <parent link="base_link"/>
         <child link="lidar_frame"/>
-        <origin xyz="0.1263 0.045 0" rpy="0 0 0"/>
+        <origin xyz="0.09 0 0" rpy="0 0 0"/>
     </joint>
     <link name="lidar_frame">

File: wallbe/description/robot_core.urdf.xacro (robot description, xacro)
@@ -6,5 +6,5 @@
   <xacro:property name="base_width" value="0.24" />
   <xacro:property name="base_length" value="0.18" />
-  <xacro:property name="base_height" value="0.056" />
+  <xacro:property name="base_height" value="0.064" />
   <xacro:property name="wheel_mass" value="0.3" /> <!-- arbitrary value for wheel mass -->
   <xacro:property name="wheel_len" value="0.024" />
